File: hardware/slushengine_modelx.kicad_pcb (KiCad board)
At the start: 2 copper layers, 261 x 100 mm, 221 parts, among them J1001 UEXT1, J12001 Stepper Motor, J13001 Stepper Motor, J14001 Stepper Motor, J2001 Stepper Motor, P1001 CONN_01X02, P1002 CONN_01X02, P1003 Raspberry_Pi_+_Conn, P1004 CONN_01X06, P1005 CONN_01X08, P1006 CONN_01X08, P1007 TST, P1008 TST, P1009 TST, P1010 TST, P1011 TST, P1012 TST, P1013 TST, P1014 TST, P1015 TST, P1016 TST, P1017 TST, P1018 TST, P1019 TST, P1020 TST, P1021 TST, P1022 TST, P1023 TST, P1024 TST, P1025 TST, P1026 TST, P1027 TST, P1028 TST, P1029 TST, P1030 TST, P1031 TST, P1032 CONN_01X06, P1033 CONN_01X06, P1034 CONN_01X06, P1035 CONN_01X03, P1036 CONN_01X02, P12001 CONN_01X04, P13001 CONN_01X04, P14001 CONN_01X04, P2001 CONN_01X04, Q10001 BCP51, Q11001 DMG2305, Q3001 BCP51, Q8001 BCP51, Q9001 BCP51, U1001 CAT24C32HU4I-GT3, U1002 LM3489, U1003 FDC5614P, U1004 LM1117IMPX-ADJ, U1005 MCP23017, U1006 MAX1164x, U11001 DMMT5401, U12001 L6470, U13001 L6470, U14001 L6470, U2001 L6470

Commit message: fixed pour issue by removing chamfers
Parts:
- added R1016: 3.9k, w_smd_resistors:r_0402, F.Cu at (-65.4, 58.5)
- added R1017: 3.9k, w_smd_resistors:r_0402, F.Cu at (-64.0, 58.5)
- R1013: value 360 -> 316
- moved C1001 316.1 mm to (-168.3, 45.4)
- moved C1002 316.1 mm to (-179.2, 54.2)
- moved C1004 316.1 mm to (-175.1, 56.6)
- moved C1005 316.1 mm to (-174.3, 62.8)
- moved C1006 316.1 mm to (-156.4, 57.5)
- moved C1007 316.1 mm to (-145.2, 43.9)
- moved C1008 316.1 mm to (-128.9, 62.5)
- moved C1009 316.1 mm to (-147.2, 64.7)
- moved C101 316.1 mm to (-245.0, 123.8)
- moved C1010 316.1 mm to (-145.1, 61.1)
- moved C12001 316.1 mm to (-152.9, 78.3)
- moved C12002 316.1 mm to (-152.8, 82.2)
- moved C12003 316.1 mm to (-151.8, 109.2)
- moved C12004 316.1 mm to (-153.8, 114.0)
- moved C12005 316.1 mm to (-157.9, 80.5)
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Routing:
- net /PI_I2C_SDA: track 405.1 -> 415.5 mm, vias 5 -> 7
- net +3V3: track 834.0 -> 839.3 mm, vias 25 -> 26
- net /PI_I2C_SCL: track 406.6 -> 410.9 mm
- net GND: track 1693.2 -> 1695.7 mm

Commit message: small board changes
Parts:
- R1014, R1015: value 50k -> 51k
- moved G*** 315.0 mm to (111.5, 134.4)
- moved C1002 311.3 mm to (132.1, 62.0)
- moved C1004 311.3 mm to (136.2, 64.5)
- moved C1007 311.3 mm to (166.1, 51.6)
- moved C1009 311.3 mm to (164.1, 72.5)
- moved C1010 311.3 mm to (166.2, 69.0)
- moved C12006 311.3 mm to (161.2, 93.5)
- moved C2006 311.3 mm to (128.7, 93.5)
- moved C4001 311.3 mm to (259.4, 118.8)
- moved C5001 311.3 mm to (259.4, 113.8)
- moved C6001 311.3 mm to (259.4, 108.8)
- moved C7001 311.3 mm to (259.4, 103.8)
- moved D1001 311.3 mm to (154.7, 58.4)
- moved D1002 311.3 mm to (166.1, 55.9)
- moved D1004 311.3 mm to (171.6, 51.7)
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Other:
- board text added: "1"
- board text added: "2"
- board text added: "B-"

Commit message: initial commit of contrib file
Routing:
- net +24V: track 545.4 -> 684.5 mm
- net GND: track 1695.7 -> 1692.0 mm
- net +3V3: track 839.3 -> 842.2 mm
- net /Stepper Driver #1/SWITCH: track 263.2 -> 261.2 mm
- net /Stepper Driver #0/SWITCH: track 301.8 -> 300.2 mm
- net /Stepper Driver #0/~STBY/RST: track 623.0 -> 624.6 mm
- net /Stepper Driver #0/SCK: track 555.9 -> 557.0 mm
- net /Stepper Driver #0/SDO: track 563.9 -> 565.0 mm
- net /Stepper Driver #2/~CS: track 251.5 -> 252.5 mm
- net /Stepper Driver #0/SDI: track 575.6 -> 576.6 mm
- net /Stepper Driver #2/SWITCH: track 221.2 -> 220.4 mm
- net /Stepper Driver #0/ADCIN: track 494.3 -> 495.1 mm
- net /Stepper Driver #2/~BUSY~/SYNC: track 261.5 -> 260.8 mm
